Commit message: test

File: urdf/urdf_assembly_2.xacro (robot description, xacro)
@@ -1,7 +1,7 @@
 <?xml version="1.0" ?>
 <robot name="urdf_assembly_2" xmlns:xacro="http://www.ros.org/wiki/xacro">
-<xacro:include filename="$(find urdf_assembly_2_description)/urdf/materials.xacro" />
-<xacro:include filename="$(find urdf_assembly_2_description)/urdf/urdf_assembly_2.trans" />
-<xacro:include filename="$(find urdf_assembly_2_description)/urdf/urdf_assembly_2.gazebo" />
+<xacro:include filename="materials.xacro" />
+<xacro:include filename="urdf_assembly_2.trans" />
+<xacro:include filename="urdf_assembly_2.gazebo" />
 <link name="base_link">
   <inertial>
@@ -13,5 +13,5 @@
     <origin xyz="0 0 0" rpy="0 0 0"/>
     <geometry>
-      <mesh filename="package://urdf_assembly_2_description/meshes/base_link.stl" scale="0.001 0.001 0.001"/>
+      <mesh filename="meshes/base_link.stl" scale="0.001 0.001 0.001"/>
     </geometry>
     <material name="silver"/>
@@ -20,5 +20,5 @@
     <origin xyz="0 0 0" rpy="0 0 0"/>
     <geometry>
-      <mesh filename="package://urdf_assembly_2_description/meshes/base_link.stl" scale="0.001 0.001 0.001"/>
+      <mesh filename="meshes/base_link.stl" scale="0.001 0.001 0.001"/>
     </geometry>
   </collision>
@@ -33,5 +33,5 @@
     <origin xyz="0.002859 0.005179 0.00232" rpy="0 0 0"/>
     <geometry>
-      <mesh filename="package://urdf_assembly_2_description/meshes/link_1_1.stl" scale="0.001 0.001 0.001"/>
+      <mesh filename="meshes/link_1_1.stl" scale="0.001 0.001 0.001"/>
     </geometry>
     <material name="silver"/>
@@ -40,5 +40,5 @@
     <origin xyz="0.002859 0.005179 0.00232" rpy="0 0 0"/>
     <geometry>
-      <mesh filename="package://urdf_assembly_2_description/meshes/link_1_1.stl" scale="0.001 0.001 0.001"/>
+      <mesh filename="meshes/link_1_1.stl" scale="0.001 0.001 0.001"/>
     </geometry>
   </collision>
@@ -53,5 +53,5 @@
     <origin xyz="0.002859 0.005179 -0.13368" rpy="0 0 0"/>
     <geometry>
-      <mesh filename="package://urdf_assembly_2_description/meshes/link_2_1.stl" scale="0.001 0.001 0.001"/>
+      <mesh filename="meshes/link_2_1.stl" scale="0.001 0.001 0.001"/>
     </geometry>
     <material name="silver"/>
@@ -60,5 +60,5 @@
     <origin xyz="0.002859 0.005179 -0.13368" rpy="0 0 0"/>
     <geometry>
-      <mesh filename="package://urdf_assembly_2_description/meshes/link_2_1.stl" scale="0.001 0.001 0.001"/>
+      <mesh filename="meshes/link_2_1.stl" scale="0.001 0.001 0.001"/>
     </geometry>
   </collision>
@@ -73,5 +73,5 @@
     <origin xyz="0.002698 0.005179 -0.432846" rpy="0 0 0"/>
     <geometry>
-      <mesh filename="package://urdf_assembly_2_description/meshes/link_3_1.stl" scale="0.001 0.001 0.001"/>
+      <mesh filename="meshes/link_3_1.stl" scale="0.001 0.001 0.001"/>
     </geometry>
     <material name="silver"/>
@@ -80,5 +80,5 @@
     <origin xyz="0.002698 0.005179 -0.432846" rpy="0 0 0"/>
     <geometry>
-      <mesh filename="package://urdf_assembly_2_description/meshes/link_3_1.stl" scale="0.001 0.001 0.001"/>
+      <mesh filename="meshes/link_3_1.stl" scale="0.001 0.001 0.001"/>
     </geometry>
   </collision>
@@ -93,5 +93,5 @@
     <origin xyz="-0.057302 0.005179 -0.530733" rpy="0 0 0"/>
     <geometry>
-      <mesh filename="package://urdf_assembly_2_description/meshes/link_4_1.stl" scale="0.001 0.001 0.001"/>
+      <mesh filename="meshes/link_4_1.stl" scale="0.001 0.001 0.001"/>
     </geometry>
     <material name="silver"/>
@@ -100,5 +100,5 @@
     <origin xyz="-0.057302 0.005179 -0.530733" rpy="0 0 0"/>
     <geometry>
-      <mesh filename="package://urdf_assembly_2_description/meshes/link_4_1.stl" scale="0.001 0.001 0.001"/>
+      <mesh filename="meshes/link_4_1.stl" scale="0.001 0.001 0.001"/>
     </geometry>
   </collision>
@@ -113,5 +113,5 @@
     <origin xyz="-0.274302 0.005096 -0.530663" rpy="0 0 0"/>
     <geometry>
-      <mesh filename="package://urdf_assembly_2_description/meshes/link_5_1.stl" scale="0.001 0.001 0.001"/>
+      <mesh filename="meshes/link_5_1.stl" scale="0.001 0.001 0.001"/>
     </geometry>
     <material name="silver"/>
@@ -120,5 +120,5 @@
     <origin xyz="-0.274302 0.005096 -0.530663" rpy="0 0 0"/>
     <geometry>
-      <mesh filename="package://urdf_assembly_2_description/meshes/link_5_1.stl" scale="0.001 0.001 0.001"/>
+      <mesh filename="meshes/link_5_1.stl" scale="0.001 0.001 0.001"/>
     </geometry>
   </collision>
@@ -133,5 +133,5 @@
     <origin xyz="-0.391802 0.005096 -0.530663" rpy="0 0 0"/>
     <geometry>
-      <mesh filename="package://urdf_assembly_2_description/meshes/link_6_1.stl" scale="0.001 0.001 0.001"/>
+      <mesh filename="meshes/link_6_1.stl" scale="0.001 0.001 0.001"/>
     </geometry>
     <material name="silver"/>
@@ -140,5 +140,5 @@
     <origin xyz="-0.391802 0.005096 -0.530663" rpy="0 0 0"/>
     <geometry>
-      <mesh filename="package://urdf_assembly_2_description/meshes/link_6_1.stl" scale="0.001 0.001 0.001"/>
+      <mesh filename="meshes/link_6_1.stl" scale="0.001 0.001 0.001"/>
     </geometry>
   </collision>
@@ -153,5 +153,5 @@
     <origin xyz="-0.396802 0.005096 -0.530663" rpy="0 0 0"/>
     <geometry>
-      <mesh filename="package://urdf_assembly_2_description/meshes/link_7_1.stl" scale="0.001 0.001 0.001"/>
+      <mesh filename="meshes/link_7_1.stl" scale="0.001 0.001 0.001"/>
     </geometry>
     <material name="silver"/>
@@ -160,5 +160,5 @@
     <origin xyz="-0.396802 0.005096 -0.530663" rpy="0 0 0"/>
     <geometry>
-      <mesh filename="package://urdf_assembly_2_description/meshes/link_7_1.stl" scale="0.001 0.001 0.001"/>
+      <mesh filename="meshes/link_7_1.stl" scale="0.001 0.001 0.001"/>
     </geometry>
   </collision>
